File: EnvFilterPedal.kicad_pcb (KiCad board)
At the start: 2 copper layers, 85 x 53 mm, 109 parts, among them J101 ScopeGroundLoop, J102 IO, Q101 BC857, Q102 BC857, U101 TL074, U102 TL074, U103 LM13700, U104 LM13700, U105 AZ34063U

Commit message: rev2 simulation stuff
Parts:
- C111, C113, C119, C120: value 1u -> 470n
- R103: value 470 -> 22k
- R110, R111: value 15k -> 6k8
- R121, R122, R124, R125: value 1k -> 680
- R130: value 4k7 -> 1k8
Changed lines of the file:
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@@
 			)
 		)
-		(property "Value" "1k"
+		(property "Value" "680"
 			(at 0 -1.65 0)
 			(layer "B.Fab")
@@
 			)
 		)
-		(property "Value" "1k"
+		(property "Value" "680"
 			(at 0 -1.65 0)
 			(layer "B.Fab")
@@
 			)
 		)
-		(property "Value" "1u"
+		(property "Value" "470n"
 			(at 0 -1.68 0)
 			(layer "B.Fab")
@@
 			)
 		)
-		(property "Value" "1u"
+		(property "Value" "470n"
 			(at 0 -1.679999 0)
 			(layer "B.Fab")
@@
 			)
 		)
-		(property "Value" "470"
+		(property "Value" "22k"
 			(at 0 -1.65 90)
 			(layer "B.Fab")
@@
 			)
 		)
-		(property "Value" "15k"
+		(property "Value" "6k8"
 			(at 0 -1.65 90)
 			(layer "B.Fab")
@@
 			)
 		)
-		(property "Value" "4k7"
+		(property "Value" "1k8"
 			(at 0 -1.65 0)
 			(layer "B.Fab")
@@
 			)
 		)
-		(property "Value" "15k"
+		(property "Value" "6k8"
 			(at 0 -1.65 90)
 			(layer "B.Fab")
@@
 			)
 		)
-		(property "Value" "1u"
+		(property "Value" "470n"
 			(at 0 -1.68 0)
 			(layer "B.Fab")
@@
 			)
 		)
-		(property "Value" "1u"
+		(property "Value" "470n"
 			(at 0 -1.679999 0)
 			(layer "B.Fab")
@@
 			)
 		)
-		(property "Value" "1k"
+		(property "Value" "680"
 			(at 0 -1.65 0)
 			(layer "B.Fab")
@@
 			)
 		)
-		(property "Value" "1k"
+		(property "Value" "680"
 			(at 0 -1.65 0)
 			(layer "B.Fab")

Commit message: 4 layer layout
Parts:
- removed R144: 33k, Resistor_SMD:R_0805_2012Metric
- removed R145, R146, R151: 100k, Resistor_SMD:R_0805_2012Metric
- removed R147: 470, Resistor_SMD:R_0805_2012Metric
- removed RV106: 100kA, Potentiometer_THT:Potentiometer_Alpha_RV16AF_42_VeryLong
- added C126: 100n, Capacitor_SMD:C_0805_2012Metric, B.Cu at (68.8, 79.2)
- added C127: 22u, Capacitor_SMD:C_0805_2012Metric, F.Cu at (78.1, 93.8)
- added D109: 1N4148W, Diode_SMD:D_SOD-123, B.Cu at (68.2, 58.0)
- added D110: 1N4148W, Diode_SMD:D_SOD-123, B.Cu at (72.1, 58.0)
- added FB101: 90R, Inductor_SMD:L_0805_2012Metric, F.Cu at (69.1, 71.5)
- added Q103: BC847, Package_TO_SOT_SMD:SOT-23, B.Cu at (22.9, 73.8)
- added TP109: +9, TestPoint:TestPoint_THTPad_D2.0mm_Drill1.0mm_VAL, F.Cu at (50.2, 84.8)
- added TP110: -9, TestPoint:TestPoint_THTPad_D2.0mm_Drill1.0mm_VAL, F.Cu at (68.1, 75.2)
- C105: value 100n -> 470u; footprint Capacitor_SMD:C_0805_2012Metric -> Capacitor_THT:CP_Radial_D5.0mm_P2.00mm
- C109: value 100n -> 1u
- C110: value 1n -> 10n
- C111: value 470n -> 100n
- C112: value 1n -> 100n
- C113, C119, C120: value 470n -> 1u
- C116: value 1u -> 1n
- C118: value 1n -> 1u
- C125: value 10n -> 1u
- D104: value 1N4148W -> LED; footprint Diode_SMD:D_SOD-123 -> LED_THT:LED_D3.0mm; moved to F.Cu
- D105, D106: value 1N4148W -> LED; footprint Diode_SMD:D_SOD-123 -> LED_THT:LED_D3.0mm
- R101, R103, R118: value 22k -> 100k
- R102: value 47k -> 100k
- R106, R125: value 680 -> 1k
- R109: value 22k -> 6k8
- R117: value 4k7 -> 100k
- R119: value 33k -> 1k8
- R120: value 33k -> 100k
- R121: value 680 -> 1M
- R122: value 680 -> 47k
- R123: value 33k -> 12k
- R124: value 680 -> 100k
- R126: value 4k7 -> 1k
- R128, R132: value 22k -> 33k
- R129: value 10k -> 1k
- R130: value 1k8 -> 1k
- R131: value 4k7 -> 33k
- R133: value 33k -> 4k7
- R134: value 1k -> 4k7
- R135: value 1k -> 10k
- R136: value 1k -> 1k8
- R137: value 1k -> 470k
- R138: value 33k -> 1Meg
- R139: value 4k7 -> 470k
- R140: value 22k -> 1Meg
- R143: value 33k -> 220
- R154: moved to B.Cu
- RV104: value 10kB -> 100kB
- RV105: value 100kB -> 100kA
- TP103: value HP -> CE
- TP104: value LP -> WET
- TP107: value HC -> GG; moved to F.Cu
- U103: value LM13700 -> TL074; footprint Package_SO:SOIC-16_3.9x9.9mm_P1.27mm -> Package_SO:SOIC-14_3.9x8.7mm_P1.27mm
- moved R138 74.9 mm to (10.4, 92.6)
- moved R148 74.8 mm to (81.0, 92.9), turned to 0 degrees
- moved C124 73.8 mm to (80.2, 73.6), turned to -90 degrees
- moved R137 72.2 mm to (13.4, 91.6)
- moved U105 71.2 mm to (78.8, 88.0), turned to -90 degrees
- moved L101 70.8 mm to (78.6, 80.6), turned to 90 degrees
- moved R140 65.9 mm to (11.8, 81.2)
- moved R150 63.1 mm to (74.2, 89.1), turned to 180 degrees
- moved C122 61.8 mm to (74.7, 86.1)
- moved D107 61.7 mm to (73.8, 81.5), turned to -90 degrees
- moved C121 60.9 mm to (66.4, 51.3), turned to -90 degrees
- moved C123 60.9 mm to (74.4, 73.8), turned to -90 degrees
- moved R149 60.1 mm to (73.9, 92.5), turned to 180 degrees
- moved R139 56.6 mm to (27.6, 87.9), turned to 180 degrees
- moved R120 55.3 mm to (10.2, 56.3), turned to 180 degrees
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Connections:
- C104 pad 1: /EnvCap -> Net-(U101C--)
- C105 pad 1: +9V -> GND
- C105 pad 2: GND -> -9V
- C106 pad 1: -9V -> +9V
- C108 pad 1: +9V -> -9V
- C109 pad 1: -9V -> FX_IN
- C109 pad 2: GND -> Net-(U103B-+)
- C110 pad 1: Net-(C110-Pad1) -> Net-(U101D-+)
- C110 pad 2: Net-(D105-A) -> GND
- C111 pad 1: Net-(C111-Pad1) -> +9V
- C111 pad 2: Net-(C111-Pad2) -> GND
- C112 pad 1: Net-(C112-Pad1) -> -9V
- C113 pad 1: Net-(C113-Pad1) -> /GTR_GAIN
- C113 pad 2: LP_OUT -> Net-(C113-Pad2)
- C116 pad 1: FX_IN -> Net-(U103D-+)
- C116 pad 2: Net-(C116-Pad2) -> GND
- C117 pad 1: Net-(C117-Pad1) -> Net-(U103A-+)
- C117 pad 2: FX_IN -> Net-(D105-A)
- C118 pad 2: /HP1 -> Net-(C118-Pad2)
- C119 pad 2: /HP1 -> Net-(C119-Pad2)
- C120 pad 2: HP_OUT -> Net-(C120-Pad2)
- C122 pad 2: -9V -> Net-(D107-A)
- C123 pad 2: -9V -> Net-(D107-A)
- C124 pad 2: -9V -> Net-(D107-A)
- C125 pad 1: Net-(U101B-+) -> -9V
- D101 pad 1: GND -> Net-(D101-K)
- D101 pad 2: /HardClip -> Net-(D101-A)
- D102 pad 1: /HardClip -> Net-(D101-A)
- D102 pad 2: GND -> Net-(D102-A)
- D103 pad 1: /FullRect -> Net-(D103-K)
- D104 pad 2: Net-(D104-A) -> +9V
- D107 pad 2: -9V -> Net-(D107-A)
- R101 pad 1: Net-(C103-Pad2) -> Net-(D102-A)
- R101 pad 2: Net-(U101A--) -> Net-(U101B--)
- R102 pad 1: Net-(U101A--) -> Net-(D102-A)
- R102 pad 2: Net-(R102-Pad2) -> Net-(U101B--)
- R103 pad 1: Net-(R103-Pad1) -> Net-(U101B--)
- R103 pad 2: /HardClip -> /FullRect
- R104 pad 1: /HardClip -> Net-(C103-Pad2)
- R104 pad 2: Net-(U101D--) -> Net-(D101-K)
- R105 pad 1: Net-(U101D--) -> Net-(D101-K)
- R105 pad 2: /FullRect -> Net-(D102-A)
- R106 pad 1: Net-(D104-K) -> Net-(D103-K)
- R106 pad 2: /EnvCap -> Net-(U101C--)
- R107 pad 1: /EnvCap -> Net-(U101C--)
- R108 pad 1: Net-(U101B--) -> Net-(U101D--)
- R108 pad 2: ENV -> /EnvPos
- R109 pad 1: Net-(U101B--) -> Net-(U101D--)
- R112 pad 1: Net-(R112-Pad1) -> ENV
- R117 pad 1: Net-(R117-Pad1) -> /EnvPos
- R117 pad 2: Iabc -> Net-(U102B--)
- R118 pad 1: Net-(C111-Pad1) -> Net-(U102B--)
- R118 pad 2: -9V -> /EnvNeg
- R119 pad 1: Net-(U103C--) -> Net-(Q103-E)
- R119 pad 2: Net-(C111-Pad2) -> GND
- R120 pad 1: Net-(C116-Pad2) -> Net-(C103-Pad2)
- R120 pad 2: Net-(U103C--) -> Net-(U101B--)
- R121 pad 1: GND -> Net-(U103B-+)
- R121 pad 2: Net-(U103C--) -> GND
- R122 pad 1: GND -> Net-(U103B--)
- R122 pad 2: Net-(U103C-+) -> /GTR_GAIN
- R123 pad 1: Net-(C111-Pad2) -> Net-(U103B--)
- R123 pad 2: Net-(U103A--) -> GND
- R124 pad 1: GND -> Net-(U101C--)
- R124 pad 2: Net-(U103A--) -> Net-(U101D-+)
- R125 pad 2: Net-(U103A-+) -> Net-(U104A--)
- R126 pad 1: Net-(R126-Pad1) -> GND
- R126 pad 2: Iabc -> Net-(U104A-+)
- R127 pad 1: Net-(U103A--) -> Net-(C113-Pad2)
- R127 pad 2: LP_OUT -> Net-(U104A--)
- R128 pad 1: Net-(C113-Pad1) -> Net-(U104A--)
- R128 pad 2: -9V -> Net-(U103A--)
- R129 pad 1: Net-(D105-A) -> GND
- R129 pad 2: Net-(D105-K) -> Net-(U104C--)
- R130 pad 1: Net-(D105-K) -> GND
- R130 pad 2: GND -> Net-(U104C-+)
- R131 pad 1: Iabc -> Net-(U103A--)
- R131 pad 2: Net-(R131-Pad2) -> Net-(U104C-+)
- R132 pad 1: Net-(C119-Pad1) -> Net-(U104C--)
- R132 pad 2: -9V -> /WET
- R133 pad 1: Net-(U104A--) -> Iabc
- R133 pad 2: /HP1 -> Net-(R133-Pad2)
- R134 pad 1: GND -> Iabc
- R134 pad 2: Net-(U104A-+) -> Net-(R134-Pad2)
- R135 pad 1: GND -> Net-(D105-A)
- R135 pad 2: Net-(U104A--) -> Net-(D105-K)
- R136 pad 2: Net-(U104C--) -> Net-(D105-K)
- R137 pad 1: GND -> Net-(C119-Pad2)
- R137 pad 2: Net-(U104C-+) -> Net-(U102A-+)
- R138 pad 1: Net-(U104C--) -> Net-(U102A-+)
- R138 pad 2: HP_OUT -> GND
- R139 pad 1: Iabc -> Net-(C118-Pad2)
- R139 pad 2: Net-(R139-Pad2) -> Net-(U102A--)
- R140 pad 1: Net-(C120-Pad1) -> Net-(U102A--)
- R140 pad 2: -9V -> Net-(R140-Pad2)
- R141 pad 1: HP_OUT -> /WET
- R141 pad 2: Net-(R141-Pad2) -> Net-(C119-Pad1)
- R142 pad 1: LP_OUT -> /GTR_GAIN
- R142 pad 2: Net-(R142-Pad2) -> Net-(C118-Pad1)
- R143 pad 1: Net-(R141-Pad2) -> Net-(C120-Pad1)
- R143 pad 2: Net-(U102C--) -> FX_OUT
- R150 pad 2: -9V -> Net-(D107-A)
- RV101 pad 1: Net-(R102-Pad2) -> GND
- RV101 pad 2: Net-(R103-Pad1) -> Net-(U103C-+)
- RV101 pad 3: Net-(R103-Pad1) -> /WET
- RV103 pad 1: GND -> /EnvNeg
- RV103 pad 2: Net-(R112-Pad1) -> ENV
- RV103 pad 3: ENV -> /EnvPos
- RV104 pad 1: GND -> Net-(C119-Pad1)
- RV104 pad 2: Net-(U102D-+) -> GND
- RV104 pad 3: LP_OUT -> Net-(C118-Pad1)
- RV105 pad 1: Net-(R141-Pad2) -> GND
- RV105 pad 2: GND -> Net-(C120-Pad2)
- RV105 pad 3: Net-(R142-Pad2) -> Net-(R140-Pad2)
- TP103 pad 1: HP_OUT -> /ComEmmiter
- TP104 pad 1: LP_OUT -> /WET
- TP107 pad 1: /HardClip -> /GTR_GAIN
- U101 pad 1: Net-(R103-Pad1) -> Net-(D101-A)
- U101 pad 12: GND -> Net-(U101D-+)
- U101 pad 14: Net-(D103-A) -> /EnvPos
- U101 pad 2: Net-(U101A--) -> Net-(D101-K)
- U101 pad 5: Net-(U101B-+) -> GND
- U101 pad 7: ENV -> /FullRect
- U101 pad 8: Net-(D104-A) -> Net-(D103-A)
- U101 pad 9: /EnvCap -> Net-(U101C--)
- U102 pad 1: unconnected-(U102-Pad1) -> Net-(R140-Pad2)
- U102 pad 10: GND -> /EnvPos
- U102 pad 12: Net-(U102D-+) -> GND
- U102 pad 13: Net-(D105-K) -> Net-(Q102-C)
- U102 pad 14: Net-(D105-A) -> Net-(C107-Pad1)
- U102 pad 2: unconnected-(U102A---Pad2) -> Net-(U102A--)
- U102 pad 3: unconnected-(U102A-+-Pad3) -> Net-(U102A-+)
- U102 pad 6: Net-(Q102-C) -> Net-(U102B--)
- U102 pad 7: Net-(C107-Pad1) -> /EnvNeg
- U102 pad 9: Net-(U102C--) -> Net-(Q103-E)
- U103 pad 1: Net-(R117-Pad1) -> Net-(U103A--)
- U103 pad 10: Net-(C112-Pad1) -> Net-(U103C-+)
- U103 pad 11: +9V -> -9V
- U103 pad 12: Net-(C112-Pad1) -> Net-(U103D-+)
- U103 pad 13: Net-(U103A--) -> /WET
- U103 pad 14: Net-(U103A-+) -> /WET
- U103 pad 2: unconnected-(U103C-DIODE_BIAS-Pad2) -> Net-(U103A--)
- U103 pad 3: Net-(U103C-+) -> Net-(U103A-+)
- U103 pad 4: Net-(U103C--) -> +9V
- U103 pad 5: Net-(C110-Pad1) -> Net-(U103B-+)
- U103 pad 6: -9V -> Net-(U103B--)
- U103 pad 7: Net-(C110-Pad1) -> /GTR_GAIN
- U103 pad 8: Net-(C111-Pad1) -> Net-(D105-A)
- U103 pad 9: Net-(C113-Pad1) -> Net-(D105-K)
- U104 pad 1: Net-(R139-Pad2) -> Net-(R134-Pad2)
- U104 pad 10: Net-(C117-Pad1) -> unconnected-(U104-Pad10)
- U104 pad 12: Net-(C117-Pad1) -> Net-(U103A-+)
- U104 pad 16: Net-(R131-Pad2) -> Net-(R133-Pad2)
- U104 pad 5: Net-(C118-Pad1) -> Net-(U103D-+)
- U104 pad 7: Net-(C118-Pad1) -> unconnected-(U104-Pad7)
- U104 pad 8: Net-(C120-Pad1) -> unconnected-(U104-Pad8)
- U104 pad 9: Net-(C119-Pad1) -> unconnected-(U104-Pad9)
- U105 pad 4: -9V -> Net-(D107-A)
Routing:
- net -9V: track 265.9 -> 123.6 mm, vias 10 -> 3
- net ENV: track 74.1 -> 0.00 mm
- net HP_OUT: track 67.2 -> 0.00 mm, vias 1 -> 0
- net FX_IN: track 58.2 -> 0.00 mm, vias 1 -> 0
- net +9V: track 224.1 -> 165.9 mm, vias 8 -> 3
- net Net-(D105-A): track 55.2 -> 0.00 mm, vias 2 -> 0
- net /vBase: track 64.7 -> 10.4 mm
- net LP_OUT: track 44.2 -> 0.00 mm
- net Net-(C103-Pad2): track 40.0 -> 0.00 mm, vias 2 -> 0
- net Net-(Q103-B): track 43.8 -> 4.74 mm, vias 2 -> 0
- net Iabc: track 37.8 -> 0.00 mm
- net Net-(D107-A): track 0.00 -> 36.0 mm
- net FX_OUT: track 30.5 -> 0.00 mm, vias 1 -> 0
- net GND: track 40.0 -> 12.6 mm, vias 33 -> 8
- net /FullRect: track 24.5 -> 0.00 mm, vias 1 -> 0
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- added copper zone on In1.Cu, net GND
- added copper zone on In2.Cu, net GND
- removed copper zone on B.Cu, net GND
- removed copper zone on F.Cu, net GND
Other:
- board size 85 x 53 mm -> 80 x 52 mm
- copper layers 2 -> 4
- board text removed: "Envelope Filter"
- board text removed: "Rev 1- 1/2025 Hayden Setlik"

Commit message: routed, DRC passing
Routing:
- net ENV_IN: track 0.00 -> 91.7 mm, vias 0 -> 2
- net /GTR_GAIN: track 0.00 -> 83.9 mm, vias 0 -> 2
- net Net-(R140-Pad2): track 0.00 -> 73.1 mm, vias 0 -> 2
- net -9V: track 123.6 -> 184.9 mm, vias 3 -> 5
- net /WET: track 0.00 -> 58.1 mm, vias 0 -> 2
- net Net-(D105-A): track 0.00 -> 51.2 mm, vias 0 -> 1
- net /EnvPos: track 0.00 -> 44.7 mm
- net +9V: track 165.9 -> 208.4 mm
- net Net-(D104-K): track 0.00 -> 40.3 mm, vias 0 -> 1
- net Net-(U103D-+): track 0.00 -> 36.2 mm, vias 0 -> 2
- net Iabc: track 0.00 -> 34.3 mm, vias 0 -> 2
- net Net-(R113-Pad1): track 0.00 -> 34.0 mm
- net GND: track 12.6 -> 45.6 mm, vias 8 -> 30
- net FX_IN: track 0.00 -> 32.4 mm, vias 0 -> 1
- net Net-(U102A--): track 0.00 -> 30.7 mm
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
Commit message: MCU pinout schematic
Routing:
- net /GTR_GAIN: track 83.9 -> 83.2 mm
- added copper zone on B.Cu, net GND
- added copper zone on F.Cu, net GND
Other:
- board text added: "Envelope Filter"
- board text added: "Rev. 2- Jan 2025 Hayden Setlik"
Changed lines of the file:
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@@
 		)
 	)
+	(gr_text "Rev. 2- Jan 2025\nHayden Setlik"
+		(at 82.75 52.25 0)
+		(layer "B.SilkS")
+		(effects
+			(font
+				(size 1 1)
+				(thickness 0.1)
+			)
+			(justify left bottom mirror)
+		)
+	)
+	(gr_text "Envelope Filter"
+		(at 83.1 49.2 0)
+		(layer "B.SilkS")
+		(effects
+			(font
+				(face "Bebas Neue")
+				(size 2.5 2.5)
+				(thickness 0.1)
+			)
+			(justify left bottom mirror)
+		)
+		(render_cache "Envelope Filter" 0
+			(polygon
+				(pts
+					(xy 82.956507 48.775) (xy 81.906873 48.775) (xy 81.906873 48.425122) (xy 82.571824 48.425122) (xy 82.571824 47.67957)
+					(xy 82.043039 47.67957) (xy 82.043039 47.329082) (xy 82.571824 47.329082) (xy 82.571824 46.66352)
+					(xy 81.906873 46.66352) (xy 81.906873 46.313032) (xy 82.956507 46.313032)
+				)
+			)
+			(polygon
+				(pts
+					(xy 81.686444 48.775) (xy 81.343893 48.775) (xy 81.343893 46.977983) (xy 81.336566 46.977983) (xy 80.874947 48.775)
+					(xy 80.479274 48.775) (xy 80.479274 46.313032) (xy 80.822435 46.313032) (xy 80.822435 47.787037)
+					(xy 80.829152 47.787037) (xy 81.203454 46.313032) (xy 81.686444 46.313032)
+				)
+			)
+			(polygon
+				(pts
+					(xy 79.9224 48.775) (xy 79.411322 48.775) (xy 79.040683 46.313032) (xy 79.393614 46.313032) (xy 79.645795 48.223011)
+					(xy 79.653122 48.223011) (xy 79.904692 46.313032) (xy 80.293649 46.313032)
+				)
+			)
+			(polygon
+				(pts
+					(xy 78.855669 48.775) (xy 77.806036 48.775) (xy 77.806036 48.425122) (xy 78.470987 48.425122) (xy 78.470987 47.67957)
+					(xy 77.942201 47.67957) (xy 77.942201 47.329082) (xy 78.470987 47.329082) (xy 78.470987 46.66352)
+					(xy 77.806036 46.66352) (xy 77.806036 46.313032) (xy 78.855669 46.313032)
+				)
+			)
+			(polygon
+				(pts
+					(xy 77.585607 48.775) (xy 76.567114 48.775) (xy 76.567114 48.425122) (xy 77.200924 48.425122) (xy 77.200924 46.313032)
+					(xy 77.585607 46.313032)
+				)
+			)
+			(polygon
+				(pts
+					(xy 75.973507 46.284353) (xy 76.117298 46.325949) (xy 76.234522 46.398183) (xy 76.324381 46.499837)
+					(xy 76.386078 46.629698) (xy 76.414626 46.753078) (xy 76.424232 46.893108) (xy 76.424232 48.195533)
+					(xy 76.414626 48.335538) (xy 76.386078 48.458848) (xy 76.324381 48.588584) (xy 76.234522 48.690097)
+					(xy 76.117298 48.7622) (xy 75.973507 48.803704) (xy 75.839881 48.814078) (xy 75.706255 48.803704)
+					(xy 75.562463 48.7622) (xy 75.44524 48.690097) (xy 75.355381 48.588584) (xy 75.293683 48.458848)
+					(xy 75.265136 48.335538) (xy 75.25553 48.195533) (xy 75.25553 46.893108) (xy 75.257205 46.868684)
+					(xy 75.640212 46.868684) (xy 75.640212 48.219958) (xy 75.657777 48.344234) (xy 75.739187 48.443218)
+					(xy 75.839881 48.4642) (xy 75.964698 48.428079) (xy 76.028831 48.320833) (xy 76.039549 48.219958)
+					(xy 76.039549 46.868684) (xy 76.021985 46.744407) (xy 75.940575 46.645423) (xy 75.839881 46.624441)
+					(xy 75.715063 46.660562) (xy 75.650931 46.767808) (xy 75.640212 46.868684) (xy 75.257205 46.868684)
+					(xy 75.265136 46.753078) (xy 75.293683 46.629698) (xy 75.355381 46.499837) (xy 75.44524 46.398183)
+					(xy 75.562463 46.325949) (xy 75.706255 46.284353) (xy 75.839881 46.273953)
+				)
+			)
+			(polygon
+				(pts
+					(xy 74.996632 48.775) (xy 74.61195 48.775) (xy 74.61195 47.796807) (xy 74.429989 47.796807) (xy 74.294705 47.786838)
+					(xy 74.151379 47.746649) (xy 74.036527 47.676186) (xy 73.949968 47.576021) (xy 73.891519 47.446729)
+					(xy 73.864878 47.322707) (xy 73.856018 47.180704) (xy 73.856018 46.929134) (xy 73.857618 46.903489)
+					(xy 74.240701 46.903489) (xy 74.240701 47.20635) (xy 74.256264 47.331932) (xy 74.339996 47.431086)
+					(xy 74.429989 47.446318) (xy 74.61195 47.446318) (xy 74.61195 46.66352) (xy 74.429989 46.66352)
+					(xy 74.308919 46.696662) (xy 74.247652 46.813774) (xy 74.240701 46.903489) (xy 73.857618 46.903489)
+					(xy 73.864878 46.787131) (xy 73.891519 46.66311) (xy 73.949968 46.533817) (xy 74.036527 46.433653)
+					(xy 74.151379 46.36319) (xy 74.294705 46.323) (xy 74.429989 46.313032) (xy 74.996632 46.313032)
+				)
+			)
+			(polygon
+				(pts
+					(xy 73.645969 48.775) (xy 72.596336 48.775) (xy 72.596336 48.425122) (xy 73.261287 48.425122) (xy 73.261287 47.67957)
+					(xy 72.732501 47.67957) (xy 72.732501 47.329082) (xy 73.261287 47.329082) (xy 73.261287 46.66352)
+					(xy 72.596336 46.66352) (xy 72.596336 46.313032) (xy 73.645969 46.313032)
+				)
+			)
+			(polygon
+				(pts
+					(xy 71.816591 48.775) (xy 71.431908 48.775) (xy 71.431908 47.718649) (xy 70.934874 47.718649) (xy 70.934874 47.368161)
+					(xy 71.431908 47.368161) (xy 71.431908 46.66352) (xy 70.798098 46.66352) (xy 70.798098 46.313032)
+					(xy 71.816591 46.313032)
+				)
+			)
+			(polygon
+				(pts
+					(xy 70.612473 48.775) (xy 70.227791 48.775) (xy 70.227791 46.313032) (xy 70.612473 46.313032)
+				)
+			)
+			(polygon
+				(pts
+					(xy 69.940806 48.775) (xy 68.922313 48.775) (xy 68.922313 48.425122) (xy 69.556123 48.425122) (xy 69.556123 46.313032)
+					(xy 69.940806 46.313032)
+				)
+			)
+			(polygon
+				(pts
+					(xy 68.709211 48.775) (xy 68.324528 48.775) (xy 68.324528 46.66352) (xy 67.922138 46.66352) (xy 67.922138 46.313032)
+					(xy 69.112212 46.313032) (xy 69.112212 46.66352) (xy 68.709211 46.66352)
+				)
+			)
+			(polygon
+				(pts
+					(xy 67.737735 48.775) (xy 66.688101 48.775) (xy 66.688101 48.425122) (xy 67.353053 48.425122) (xy 67.353053 47.67957)
+					(xy 66.824267 47.67957) (xy 66.824267 47.329082) (xy 67.353053 47.329082) (xy 67.353053 46.66352)
+					(xy 66.688101 46.66352) (xy 66.688101 46.313032) (xy 67.737735 46.313032)
+				)
+			)
+			(polygon
+				(pts
+					(xy 66.467672 48.775) (xy 66.08299 48.775) (xy 66.08299 47.718649) (xy 65.949877 47.718649) (xy 65.826988 47.737989)
+					(xy 65.738795 47.825058) (xy 65.710462 47.961133) (xy 65.708688 48.02151) (xy 65.708688 48.472138)
+					(xy 65.706159 48.595367) (xy 65.690956 48.71735) (xy 65.673272 48.775) (xy 65.281263 48.775) (xy 65.314374 48.653924)
+					(xy 65.323007 48.529711) (xy 65.323394 48.475802) (xy 65.323394 48.042271) (xy 65.328255 47.919124)
+					(xy 65.348393 47.790671) (xy 65.394939 47.668856) (xy 65.48365 47.568784) (xy 65.578628 47.522644)
+					(xy 65.578628 47.515317) (xy 65.467192 47.445822) (xy 65.388729 47.341752) (xy 65.346402 47.222328)
+					(xy 65.329191 47.098894) (xy 65.327058 47.029884) (xy 65.327058 46.916922) (xy 65.711741 46.916922)
+					(xy 65.711741 47.107431) (xy 65.727721 47.231633) (xy 65.79796 47.332191) (xy 65.916915 47.367406)
+					(xy 65.943161 47.368161) (xy 66.08299 47.368161) (xy 66.08299 46.66352) (xy 65.907745 46.66352)
+					(xy 65.78589 46.69733) (xy 65.723218 46.803139) (xy 65.711741 46.916922) (xy 65.327058 46.916922)
+					(xy 65.327058 46.878454) (xy 65.335209 46.745115) (xy 65.369011 46.603888) (xy 65.430236 46.490751)
+					(xy 65.520156 46.405511) (xy 65.640042 46.34797) (xy 65.791167 46.317933) (xy 65.897365 46.313032)
+					(xy 66.467672 46.313032)
+				)
+			)
+		)
+	)
 	(gr_text "OUT"
 		(at 39.3 91.2 -90)
@@
 	)
 	(segment
-		(start 56.55 56.75)
-		(end 58.7 54.6)
+		(start 59.9 54.6)
+		(end 60.7 54.6)
 		(width 0.18)
 		(layer "F.Cu")
@@
 	)
 	(segment
-		(start 58.7 54.6)
-		(end 60.7 54.6)
+		(start 56.55 66.95)
+		(end 56.55 57.95)
 		(width 0.18)
 		(layer "F.Cu")
@@
 	)
 	(segment
-		(start 56.55 66.95)
-		(end 56.55 56.75)
+		(start 56.55 57.95)
+		(end 59.9 54.6)
 		(width 0.18)
 		(layer "F.Cu")
@@
 	)
 	(segment
-		(start 27.15 71.45)
-		(end 27.675 70.925)
+		(start 24.975 70.925)
+		(end 32.725 70.925)
 		(width 0.18)
 		(layer "F.Cu")
@@
 	)
 	(segment
-		(start 20.9875 71.45)
-		(end 27.15 71.45)
+		(start 18.075 68.5375)
+		(end 20.9875 71.45)
 		(width 0.18)
 		(layer "F.Cu")
@@
 	)
 	(segment
-		(start 27.675 70.925)
-		(end 32.725 70.925)
+		(start 20.9875 71.45)
+		(end 24.45 71.45)
 		(width 0.18)
 		(layer "F.Cu")
@@
 	)
 	(segment
-		(start 18.075 68.5375)
-		(end 20.9875 71.45)
+		(start 24.45 71.45)
+		(end 24.975 70.925)
 		(width 0.18)
 		(layer "F.Cu")
@@
 	)
 	(zone
+		(net 1)
+		(net_name "GND")
+		(locked yes)
+		(layers "F&B.Cu")
+		(hatch edge 0.5)
+		(priority 1)
+		(connect_pads
+			(clearance 0.25)
+		)
+		(min_thickness 0.25)
+		(filled_areas_thickness no)
+		(fill yes
+			(thermal_gap 0.5)
+			(thermal_bridge_width 0.5)
+		)
+		(polygon
+			(pts
+				(xy 5 96.5) (xy 4.5 96) (xy 4.5 45) (xy 83.5 45) (xy 83.5 96.5)
+			)
+		)
+	)
+	(zone

Commit message: cleaned up routing
Parts:
- moved TP105 5.25 mm to (28.4, 68.0)
- moved R110 1.80 mm to (53.4, 47.5), turned to -90 degrees
Routing:
- net Net-(U102A--): track 30.7 -> 20.4 mm, vias 0 -> 2
- net Net-(D104-K): track 40.3 -> 35.6 mm
- net +9V: track 208.4 -> 204.0 mm
- net /EnvPos: track 44.7 -> 47.4 mm
- net Net-(R110-Pad2): track 2.81 -> 4.50 mm
- net ENV: track 20.0 -> 21.0 mm
- net Net-(C119-Pad1): track 24.4 -> 25.2 mm, vias 1 -> 0

Commit message: rev2 gerber
Parts:
- added TP111: LP1, TestPoint:TestPoint_THTPad_D2.0mm_Drill1.0mm_VAL, F.Cu at (35.6, 65.0)
- added TP112: LP2, TestPoint:TestPoint_THTPad_D2.0mm_Drill1.0mm_VAL, F.Cu at (68.5, 63.6)
- added TP113: FB, TestPoint:TestPoint_THTPad_D2.0mm_Drill1.0mm_VAL, F.Cu at (46.2, 82.8)
- moved J101 27.1 mm to (61.7, 84.0)
Connections:
- net Net-(D105-A) renamed /Feedback
- net Net-(U103A-+) renamed /LP1
- net Net-(U103D-+) renamed /LP2
Routing:
- net /LP1: track 27.7 -> 46.1 mm
- net Net-(U101B--): track 22.1 -> 35.9 mm
- net /Feedback: track 51.2 -> 60.5 mm
- net +9V: track 204.0 -> 199.0 mm, vias 3 -> 4
- net /LP2: track 36.2 -> 40.5 mm
- net GND: track 45.9 -> 43.4 mm, vias 30 -> 106
- net Net-(U103C-+): track 25.4 -> 27.3 mm
- net Net-(R113-Pad1): track 34.0 -> 32.8 mm
