File: EnvFilterPedal.kicad_pcb (KiCad board)
At the start: 4 copper layers, 80 x 52 mm, 111 parts, among them J1 ScopeGroundLoop, J2 IO, Q1 BC847, Q2 BC857, Q3 BC857, U1 TL074, U2 TL074, U3 TL074, U4 LM13700, U5 AZ34063U

Commit message: rev4 sent to fab
Routing:
- net +9V: track 215.0 -> 213.0 mm, vias 3 -> 4
Changed lines of the file:
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@@
+		(net 3)
+	)
+	(via
+		(at 46.75 51.825)
+		(size 0.8)
+		(drill 0.4)
+		(layers "F.Cu" "B.Cu")
 		(net 3)
 	)
@@
 		(width 0.35)
 		(layer "B.Cu")
-		(net 3)
-	)
-	(segment
-		(start 46.75 49.875)
-		(end 46.75 51.825)
-		(width 0.35)
-		(layer "B.Cu")
