File: EnvFilterPedal.kicad_pcb (KiCad board)
At the start: 4 copper layers, 80 x 52 mm, 111 parts, among them J1 ScopeGroundLoop, J2 IO, Q1 BC847, Q2 BC857, Q3 BC857, U1 TL074, U2 TL074, U3 TL074, U4 LM13700, U5 AZ34063U

Commit message: rev5 routed & drc passing
Parts:
- removed C1, C10, C2, C3, C4, C5, C7, C8, C9: 100n, Capacitor_SMD:C_0805_2012Metric
- removed C11, C12, C18, C19, C23, C6: 1u, Capacitor_SMD:C_0805_2012Metric
- removed C13: 33n, Capacitor_SMD:C_0805_2012Metric
- removed C14, C15: 1n, Capacitor_SMD:C_0805_2012Metric
- removed C16: 4n7, Capacitor_SMD:C_0805_2012Metric
- removed C17, C21, C24: 220u, Capacitor_THT:CP_Radial_D5.0mm_P2.00mm
- removed C20: 470p, Capacitor_SMD:C_0805_2012Metric
- removed C22: 470u, Capacitor_THT:CP_Radial_D5.0mm_P2.00mm
- removed C25: 100u, Capacitor_THT:CP_Radial_D5.0mm_P2.00mm
- removed C26: 10u, Capacitor_SMD:C_0805_2012Metric
- removed D2, D3, D4, D5: 1N4148W, Diode_SMD:D_SOD-123
- removed D6, D8: LED, LED_THT:LED_D3.0mm
- removed D7: PMEG3030, Diode_SMD:D_SOD-123
- removed J1: ScopeGroundLoop, Connector_Pin:THT_GND_WIRE
- removed J2: IO, Connector_PinHeader_2.54mm:PinHeader_1x05_P2.54mm_Vertical
- removed L2: 4u7, Inductor_SMD:L_Bourns_SRP3212
- removed Q1: BC847, Package_TO_SOT_SMD:SOT-23
- removed Q2, Q3: BC857, Package_TO_SOT_SMD:SOT-23
- removed R1, R11, R14, R16, R21, R3, R32, R33, R5, R7: 100k, Resistor_SMD:R_0805_2012Metric
- removed R10, R38, R39, R6: 47k, Resistor_SMD:R_0805_2012Metric
- removed R12: 22k, Resistor_SMD:R_0805_2012Metric
- removed R13, R18, R23, R28: 33k, Resistor_SMD:R_0805_2012Metric
- removed R15, R17, R24, R27, R8: 1k, Resistor_SMD:R_0805_2012Metric
- removed R19, R29, R36: 4k7, Resistor_SMD:R_0805_2012Metric
- removed R2: 1M, Resistor_SMD:R_0805_2012Metric
- removed R20: 5k1, Resistor_SMD:R_0805_2012Metric
- removed R22, R31: 10k, Resistor_SMD:R_0805_2012Metric
- removed R25, R34: 2k2, Resistor_SMD:R_0805_2012Metric
- removed R26, R30: 6k8, Resistor_SMD:R_0805_2012Metric
- removed R35, R42, R43: 470k, Resistor_SMD:R_0805_2012Metric
- removed R37: 0.24R, Resistor_SMD:R_0805_2012Metric
- removed R4, R47: 12k, Resistor_SMD:R_0805_2012Metric
- removed R40: 51k, Resistor_SMD:R_0805_2012Metric
- removed R41: 8k2, Resistor_SMD:R_0805_2012Metric
- removed R44, R45: 1Meg, Resistor_SMD:R_0805_2012Metric
- removed R46: 220, Resistor_SMD:R_0805_2012Metric
- removed RV1, RV2: 10kB, Potentiometer_THT:Potentiometer_Alpha_RV16AF_42_Single_Long
- removed RV3, RV4: 100kB, Potentiometer_THT:Potentiometer_Alpha_RV16AF_42_Single_Long
- removed RV5: 100kA, Potentiometer_THT:Potentiometer_Alpha_RV16AF_42_Single_Long
- removed TP1: LP1, TestPoint:TestPoint_THTPad_D2.0mm_Drill1.0mm_VAL
- removed TP10: ENV, TestPoint:TestPoint_THTPad_D2.0mm_Drill1.0mm_VAL
- removed TP11: ENV_IN, TestPoint:TestPoint_THTPad_D2.0mm_Drill1.0mm_VAL
- removed TP12: +9, TestPoint:TestPoint_THTPad_D2.0mm_Drill1.0mm_VAL
- removed TP13: -9, TestPoint:TestPoint_THTPad_D2.0mm_Drill1.0mm_VAL
- removed TP14: -9R, TestPoint:TestPoint_THTPad_D2.0mm_Drill1.0mm_VAL
- removed TP2: In, TestPoint:TestPoint_THTPad_D2.0mm_Drill1.0mm_VAL
- removed TP3: LP2, TestPoint:TestPoint_THTPad_D2.0mm_Drill1.0mm_VAL
- removed TP4: Out, TestPoint:TestPoint_THTPad_D2.0mm_Drill1.0mm_VAL
- removed TP5: FR, TestPoint:TestPoint_THTPad_D2.0mm_Drill1.0mm_VAL
- removed TP6: GG, TestPoint:TestPoint_THTPad_D2.0mm_Drill1.0mm_VAL
- removed TP7: FB, TestPoint:TestPoint_THTPad_D2.0mm_Drill1.0mm_VAL
- removed TP8: CE, TestPoint:TestPoint_THTPad_D2.0mm_Drill1.0mm_VAL
- removed TP9: WET, TestPoint:TestPoint_THTPad_D2.0mm_Drill1.0mm_VAL
- removed U2, U3: TL074, Package_SO:SOIC-14_3.9x8.7mm_P1.27mm
- removed U4: LM13700, Package_SO:SOIC-16_3.9x9.9mm_P1.27mm
- removed U5: AZ34063U, Package_SO:SO-8_3.9x4.9mm_P1.27mm
- added C101: 100n, Capacitor_SMD:C_0805_2012Metric, B.Cu at (22.0, 56.2)
- added C102: 100n, Capacitor_SMD:C_0805_2012Metric, B.Cu at (10.7, 56.1)
- added C103: 1u, Capacitor_SMD:C_0805_2012Metric, B.Cu at (7.72, 68.2)
- added C104: 1u, Capacitor_SMD:C_0805_2012Metric, B.Cu at (21.3, 53.4)
- added C106: 100n, Capacitor_SMD:C_0805_2012Metric, B.Cu at (33.4, 68.4)
- added C107: 4n7, Capacitor_SMD:C_0805_2012Metric, B.Cu at (37.5, 57.6)
- added C108: 100n, Capacitor_SMD:C_0805_2012Metric, B.Cu at (33.4, 57.1)
- added C109: 1u, Capacitor_SMD:C_0805_2012Metric, B.Cu at (43.4, 84.3)
- added C110: 33n, Capacitor_SMD:C_0805_2012Metric, B.Cu at (25.0, 58.7)
- added C111: 100n, Capacitor_SMD:C_0805_2012Metric, B.Cu at (32.5, 85.2)
- added C112: 100n, Capacitor_SMD:C_0805_2012Metric, B.Cu at (32.5, 73.6)
- added C113: 1u, Capacitor_SMD:C_0805_2012Metric, B.Cu at (53.6, 82.8)
- added C114: 100n, Capacitor_SMD:C_0805_2012Metric, B.Cu at (64.6, 79.1)
- added C115: 100n, Capacitor_SMD:C_0805_2012Metric, B.Cu at (65.0, 67.4)
- added C116: 1n, Capacitor_SMD:C_0805_2012Metric, B.Cu at (36.0, 73.5)
- added C117: 1n, Capacitor_SMD:C_0805_2012Metric, B.Cu at (23.6, 79.3)
- added C118: 1u, Capacitor_SMD:C_0805_2012Metric, B.Cu at (30.4, 89.3)
- added C119: 1u, Capacitor_SMD:C_0805_2012Metric, B.Cu at (23.1, 89.5)
- added C120: 1u, Capacitor_SMD:C_0805_2012Metric, B.Cu at (63.1, 88.7)
- added C121: 100u, Capacitor_THT:CP_Radial_D5.0mm_P2.00mm, B.Cu at (57.4, 57.3)
- added C122: 100p, Capacitor_SMD:C_0805_2012Metric, B.Cu at (77.4, 79.8)
- added C123: 4u7, Capacitor_SMD:C_0805_2012Metric, B.Cu at (73.5, 79.8)
- added C124: 2u2, Capacitor_SMD:C_0805_2012Metric, B.Cu at (77.4, 93.1)
- added C125: 100u, Capacitor_THT:CP_Radial_D5.0mm_P2.00mm, B.Cu at (63.6, 57.3)
- added D101: 1N4148W, Diode_SMD:D_SOD-123, B.Cu at (11.2, 59.8)
- added D102: 1N4148W, Diode_SMD:D_SOD-123, B.Cu at (9.98, 63.5)
- added D103: 1N4148W, Diode_SMD:D_SOD-123, B.Cu at (15.7, 49.4)
- added D104: LED, LED_THT:LED_D3.0mm, F.Cu at (30.1, 48.8)
- added D108: LED, LED_THT:LED_D3.0mm, F.Cu at (56.6, 48.8)
- added D109: 1N4148W, Diode_SMD:D_SOD-123, B.Cu at (18.2, 76.1)
- added D110: 1N4148W, Diode_SMD:D_SOD-123, B.Cu at (14.3, 76.0)
- added J101: ScopeGroundLoop, Connector:THT_GND_WIRE, B.Cu at (7.20, 83.3)
- added J102: IO, Connector_PinHeader_2.54mm:PinHeader_1x05_P2.54mm_Vertical, F.Cu at (40.1, 93.0)
- added NT1: NetTie_2, NetTie:NetTie-2_SMD_Pad0.5mm, B.Cu at (70.2, 89.2)
- added Q101: BC857, Package_TO_SOT_SMD:SOT-23, B.Cu at (49.0, 58.2)
- added Q102: BC857, Package_TO_SOT_SMD:SOT-23, B.Cu at (44.8, 58.0)
- added Q103: BC847, Package_TO_SOT_SMD:SOT-23, B.Cu at (30.4, 53.1)
- added R102: 100k, Resistor_SMD:R_0805_2012Metric, B.Cu at (7.75, 51.7)
- added R103: 100k, Resistor_SMD:R_0805_2012Metric, B.Cu at (11.3, 51.7)
- added R104: 100k, Resistor_SMD:R_0805_2012Metric, B.Cu at (7.75, 59.3)
- added R105: 100k, Resistor_SMD:R_0805_2012Metric, B.Cu at (14.3, 63.5)
- added R106: 1k, Resistor_SMD:R_0805_2012Metric, B.Cu at (19.2, 49.5)
- added R107: 22k, Resistor_SMD:R_0805_2012Metric, B.Cu at (25.0, 51.2)
- added R108: 100k, Resistor_SMD:R_0805_2012Metric, B.Cu at (22.0, 62.8)
- added R109: 5k1, Resistor_SMD:R_0805_2012Metric, B.Cu at (21.9, 59.5)
- added R110: 6k8, Resistor_SMD:R_0805_2012Metric, B.Cu at (49.2, 52.7)
- added R111: 10k, Resistor_SMD:R_0805_2012Metric, B.Cu at (39.2, 52.8)
- added R112: 100k, Resistor_SMD:R_0805_2012Metric, B.Cu at (40.6, 62.3)
- added R113: 100k, Resistor_SMD:R_0805_2012Metric, B.Cu at (44.4, 52.8)
- added R114: 2k2, Resistor_SMD:R_0805_2012Metric, B.Cu at (43.8, 62.2)
- added R115: 470k, Resistor_SMD:R_0805_2012Metric, B.Cu at (40.6, 56.5)
- added R116: 4k7, Resistor_SMD:R_0805_2012Metric, B.Cu at (49.1, 61.0)
- added R117: 100k, Resistor_SMD:R_0805_2012Metric, B.Cu at (26.8, 64.2)
- added R118: 100k, Resistor_SMD:R_0805_2012Metric, B.Cu at (29.2, 68.2)
- added R119: 2k2, Resistor_SMD:R_0805_2012Metric, B.Cu at (33.4, 53.2)
- added R120: 100k, Resistor_SMD:R_0805_2012Metric, B.Cu at (7.75, 55.5)
- added R121: 1M, Resistor_SMD:R_0805_2012Metric, B.Cu at (43.6, 81.0)
- added R122: 47k, Resistor_SMD:R_0805_2012Metric, B.Cu at (37.0, 67.5)
- added R123: 12k, Resistor_SMD:R_0805_2012Metric, B.Cu at (37.0, 69.5)
- added R124: 100k, Resistor_SMD:R_0805_2012Metric, B.Cu at (25.0, 55.0)
- added R125: 1k, Resistor_SMD:R_0805_2012Metric, B.Cu at (60.3, 79.3)
- added R126: 1k, Resistor_SMD:R_0805_2012Metric, B.Cu at (57.0, 79.2)
- added R127: 33k, Resistor_SMD:R_0805_2012Metric, B.Cu at (57.6, 82.8)
- added R128: 33k, Resistor_SMD:R_0805_2012Metric, B.Cu at (39.1, 82.3)
- added R129: 1k, Resistor_SMD:R_0805_2012Metric, B.Cu at (61.4, 67.2)
- added R130: 1k, Resistor_SMD:R_0805_2012Metric, B.Cu at (58.0, 67.2)
- added R131: 33k, Resistor_SMD:R_0805_2012Metric, B.Cu at (59.5, 64.3)
- added R132: 33k, Resistor_SMD:R_0805_2012Metric, B.Cu at (40.2, 76.0)
- added R133: 4k7, Resistor_SMD:R_0805_2012Metric, B.Cu at (53.4, 76.0)
- added R134: 4k7, Resistor_SMD:R_0805_2012Metric, B.Cu at (53.6, 70.2)
- added R135: 10k, Resistor_SMD:R_0805_2012Metric, B.Cu at (28.8, 74.6)
- added R136: 6k8, Resistor_SMD:R_0805_2012Metric, B.Cu at (28.8, 72.5)
- added R137: 470k, Resistor_SMD:R_0805_2012Metric, B.Cu at (19.8, 89.5)
- added R138: 1Meg, Resistor_SMD:R_0805_2012Metric, B.Cu at (16.2, 89.5)
- added R139: 470k, Resistor_SMD:R_0805_2012Metric, B.Cu at (27.2, 89.3)
- added R140: 1Meg, Resistor_SMD:R_0805_2012Metric, B.Cu at (29.1, 85.7)
- added R141: 47k, Resistor_SMD:R_0805_2012Metric, B.Cu at (16.9, 93.0)
- added R142: 47k, Resistor_SMD:R_0805_2012Metric, B.Cu at (34.7, 93.0)
- added R143: 220, Resistor_SMD:R_0805_2012Metric, B.Cu at (59.4, 88.7)
- added R144: 300k, Resistor_SMD:R_0805_2012Metric, B.Cu at (77.4, 81.9)
- added R145: 22k, Resistor_SMD:R_0805_2012Metric, B.Cu at (77.4, 83.9)
- added R146: 47k, Resistor_SMD:R_0805_2012Metric, B.Cu at (77.4, 91.0)
- added R154: 12k, Resistor_SMD:R_0805_2012Metric, B.Cu at (58.1, 52.2)
- added RV101: 100kB, Potentiometer_THT:Potentiometer_Alpha_RV16AF_42_VeryLong, F.Cu at (69.1, 68.5)
- added RV102: 10kB, Potentiometer_THT:Potentiometer_Alpha_RV16AF_42_VeryLong, F.Cu at (39.2, 49.2)
- added RV103: 10kB, Potentiometer_THT:Potentiometer_Alpha_RV16AF_42_VeryLong, F.Cu at (13.1, 68.5)
- added RV104: 100kB, Potentiometer_THT:Potentiometer_Alpha_RV16AF_42_VeryLong, F.Cu at (20.5, 93.0)
- added RV105: 100kA, Potentiometer_THT:Potentiometer_Alpha_RV16AF_42_VeryLong, F.Cu at (57.0, 93.0)
- added TP101: In, TestPoint:TestPoint_THTPad_D2.0mm_Drill1.0mm_VAL, B.Cu at (46.9, 84.3)
- added TP102: Out, TestPoint:TestPoint_THTPad_D2.0mm_Drill1.0mm_VAL, B.Cu at (55.9, 88.8)
- added TP103: CE, TestPoint:TestPoint_THTPad_D2.0mm_Drill1.0mm_VAL, B.Cu at (49.1, 64.7)
- added TP104: WET, TestPoint:TestPoint_THTPad_D2.0mm_Drill1.0mm_VAL, B.Cu at (79.2, 63.4)
- added TP105: ENV, TestPoint:TestPoint_THTPad_D2.0mm_Drill1.0mm_VAL, B.Cu at (18.1, 65.2)
- added TP106: ENV_IN, TestPoint:TestPoint_THTPad_D2.0mm_Drill1.0mm_VAL, B.Cu at (7.74, 72.9)
- added TP107: GG, TestPoint:TestPoint_THTPad_D2.0mm_Drill1.0mm_VAL, B.Cu at (44.2, 66.6)
- added TP108: FR, TestPoint:TestPoint_THTPad_D2.0mm_Drill1.0mm_VAL, B.Cu at (11.0, 48.4)
- added TP109: +9, TestPoint:TestPoint_THTPad_D2.0mm_Drill1.0mm_VAL, B.Cu at (76.4, 76.7)
- added TP110: -9, TestPoint:TestPoint_THTPad_D2.0mm_Drill1.0mm_VAL, B.Cu at (70.4, 76.3)
- added TP111: LP1, TestPoint:TestPoint_THTPad_D2.0mm_Drill1.0mm_VAL, B.Cu at (19.8, 81.4)
- added TP112: LP2, TestPoint:TestPoint_THTPad_D2.0mm_Drill1.0mm_VAL, B.Cu at (44.0, 71.6)
- added TP113: FB, TestPoint:TestPoint_THTPad_D2.0mm_Drill1.0mm_VAL, B.Cu at (10.3, 77.6)
- added U101: TL074, Package_SO:SOIC-14_3.9x8.7mm_P1.27mm, B.Cu at (16.2, 56.2)
- added U102: TL074, Package_SO:SOIC-14_3.9x8.7mm_P1.27mm, B.Cu at (33.4, 62.7)
- added U103: TL074, Package_SO:SOIC-14_3.9x8.7mm_P1.27mm, B.Cu at (32.5, 79.3)
- added U104: LM13700, Package_SO:SOIC-16_3.9x9.9mm_P1.27mm, B.Cu at (61.2, 73.2)
- D1: value 1N4148W -> SS1060FL; footprint Diode_SMD:D_SOD-123 -> Diode_SMD:D_SOD-123F
- L1: value 68uH -> 10u; footprint Inductor_SMD:L_TDK_VLS6045EX_VLS6045AF -> Inductor_SMD:L_SigTransformer_SLPPI04_15; moved to B.Cu
- U1: value TL074 -> LMR62014XMF; footprint Package_SO:SOIC-14_3.9x8.7mm_P1.27mm -> Package_TO_SOT_SMD:SOT-23-5
- moved U1 61.9 mm to (77.4, 87.5), turned to -90 degrees
- moved D1 51.1 mm to (73.3, 82.0)
- moved L1 1.01 mm to (73.3, 87.4), turned to 90 degrees
Connections:
- D1 pad 1: Net-(D1-K) -> +9V
- L1 pad 1: /SWE -> VCC
- L1 pad 2: GND -> Net-(D1-A)
- U1 pad 2: Net-(D1-K) -> -9V
- U1 pad 3: GND -> Net-(U1-FB)
- U1 pad 4: +9V -> Net-(U1-EN)
- U1 pad 5: GND -> VCC
Routing:
- net -9V: track 234.9 -> 293.2 mm, vias 6 -> 4
- net Net-(U103C-+): track 0.00 -> 57.6 mm, vias 0 -> 1
- net Net-(R45-Pad2): track 52.6 -> 0.00 mm
- net Net-(R140-Pad2): track 0.00 -> 50.9 mm, vias 0 -> 1
- net /vBase: track 66.4 -> 20.9 mm
- net Net-(U102A-+): track 0.00 -> 42.8 mm, vias 0 -> 2
- net VCC: track 0.00 -> 38.7 mm
- net GND: track 40.2 -> 2.35 mm, vias 66 -> 54
- net Net-(U103A--): track 0.00 -> 35.5 mm, vias 0 -> 2
- net Net-(U104A--): track 0.00 -> 35.2 mm
- net FX_IN: track 41.8 -> 11.9 mm
- net Net-(C18-Pad1): track 29.4 -> 0.00 mm
- net /-9RAW: track 28.2 -> 0.00 mm
- net Net-(D102-A): track 0.00 -> 28.2 mm
- net Net-(U4A--): track 28.2 -> 0.00 mm, vias 2 -> 0
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Other:
- board text added: "Rev. 4- 07/2026 Hayden Setlik"
- board text removed: "Rev. 4- 03/2026 Hayden Setlik"
