File: EnvFilterPedal.kicad_sch (KiCad schematic)
At the start: 52 parts, among them J101 ScopeGroundLoop, J102 IO, Q101 BC857, Q102 BC857, U101 TL074, U105 AZ34063U

Commit message: rev2 schematic and footprints
Parts:
- added C106, C108, C111, C112, C114, C115, C126: 100n, Capacitor_SMD:C_0805_2012Metric, symbol Device:C
- added C109, C113, C118, C119, C120, C125: 1u, Capacitor_SMD:C_0805_2012Metric, symbol Device:C
- added C110: 10n, Capacitor_SMD:C_0805_2012Metric, symbol Device:C
- added C116, C117: 1n, Capacitor_SMD:C_0805_2012Metric, symbol Device:C
- added D104, D105, D106: LED, LED_THT:LED_D3.0mm, symbol Device:LED
- added D109, D110: 1N4148W, Diode_SMD:D_SOD-123, symbol Diode:1N4148W
- added Q103: BC847, Package_TO_SOT_SMD:SOT-23, symbol Transistor_BJT:BC847
- added R117, R118, R120, R124: 100k, Resistor_SMD:R_0805_2012Metric, symbol Device:R_US
- added R119, R136: 1k8, Resistor_SMD:R_0805_2012Metric, symbol Device:R_US
- added R121: 1M, Resistor_SMD:R_0805_2012Metric, symbol Device:R_US
- added R122, R141, R142: 47k, Resistor_SMD:R_0805_2012Metric, symbol Device:R_US
- added R123: 12k, Resistor_SMD:R_0805_2012Metric, symbol Device:R_US
- added R125, R126, R129, R130: 1k, Resistor_SMD:R_0805_2012Metric, symbol Device:R_US
- added R127, R128, R131, R132: 33k, Resistor_SMD:R_0805_2012Metric, symbol Device:R_US
- added R133, R134: 4k7, Resistor_SMD:R_0805_2012Metric, symbol Device:R_US
- added R135: 10k, Resistor_SMD:R_0805_2012Metric, symbol Device:R_US
- added R137, R139: 470k, Resistor_SMD:R_0805_2012Metric, symbol Device:R_US
- added R138, R140: 1Meg, Resistor_SMD:R_0805_2012Metric, symbol Device:R_US
- added R143: 220, Resistor_SMD:R_0805_2012Metric, symbol Device:R_US
- added RV101, RV104: 100kB, Potentiometer_THT:Potentiometer_Alpha_RV16AF_42_VeryLong, symbol Device:R_Potentiometer_US
- added RV105: 100kA, Potentiometer_THT:Potentiometer_Alpha_RV16AF_42_VeryLong, symbol Device:R_Potentiometer_US
- added U102, U103: TL074, Package_SO:SOIC-14_3.9x8.7mm_P1.27mm, symbol Amplifier_Operational:TL074
- added U104: LM13700, Package_SO:SOIC-16_3.9x9.9mm_P1.27mm, symbol Amplifier_Operational:LM13700
Connections:
- net +9V: now also C106.1, C111.1, C114.1, D104.2 (A), U102.4 (V+), U103.4 (V+), U104.11 (V+)
- net -9V: now also C108.1, C112.1, C115.1, C125.1, C126.1, U102.11 (V-), U103.11 (V-), U104.6 (V-)
- net ENV: now also R112.1, RV103.2; no longer R108.2, RV103.3, U101.7
- net FX_IN: now also C109.1
- net FX_OUT: now also R143.2
- net GND: now also C106.2, C108.2, C110.2, C111.2, C112.2, C114.2, C115.2, C116.2, C125.2, C126.2, R119.2, R121.2, R123.2, R125.1, R126.1, R129.1, R130.1, R136.1, R138.2, RV101.1, RV104.2, RV105.1, U102.3 (+), U103.9 (-); no longer RV103.1
- net Iabc: now also R133.1, R134.1
- net at C104.1, R106.2, R107.1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: now also R124.1; no longer U101.5 (+)
- net at R101.2, R102.2, R103.1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: now also R120.2
- net at C103.2, R104.1: now also R120.1
- net at C107.2, Q102.3 (C), R115.1: now also U103.10 (+)
- net at C107.1, R116.2: now also U103.8
- new net: C117.1, U103.3 (+), U104.12
- new net: C117.2, D105.2 (A), D106.1 (K), D109.2 (A), D110.1 (K), R135.1, U103.7
- new net: C110.1, R124.2, U101.5 (+)
- new net: Q103.1 (B), U102.7
- new net: Q103.2 (E), R119.1, U102.5 (+)
- new net: D104.1 (K), Q103.3 (C)
- new net: C120.2, RV105.2
- new net: R140.2, RV105.3, U102.14
- new net: D105.1 (K), D106.2 (A), D109.1 (K), D110.2 (A), R135.2, R136.2, U103.6 (-)
- new net: R122.1, R123.1, U102.9 (-)
- new net: R126.2, U104.14 (+)
- new net: C120.1, R143.1
- new net: C118.1, R142.2, RV104.3
- new net: C118.2, R139.1
- new net: R137.2, R138.1, U102.12 (+)
- new net: R139.2, R140.1, U102.13 (-)
- new net: R129.2, R132.1, U104.4 (-)
- new net: C113.2, R127.1
- new net: C109.2, R121.1, U102.10 (+)
- new net: R128.2, R131.1, U103.1, U103.2 (-)
- new net: R125.2, R127.2, R128.1, U104.13 (-)
- new net: C116.1, U103.12 (+), U104.5
- new net: R130.2, R131.2, U104.3 (+)
- new net: R134.2, U104.1
- new net: RV101.2, U103.5 (+)
- new net: C119.1, R141.2, RV104.1
- new net: R117.2, R118.1, U102.2 (-)
- new net: R133.2, U104.16
- new net: C119.2, R137.1
- new net EnvNeg: R118.2, RV103.1, U102.1
- new net EnvPos: R108.2, R117.1, RV103.3, U101.7, U102.6 (-)
- new net GTR_GAIN: C113.1, R122.2, R142.1, U102.8
- new net WET: R132.2, R141.1, RV101.3, U103.13 (-), U103.14
- no-connect marks 0 -> 5
Other:
- note added: "Envelope LED"
- note added: "Resonance"
- note added: "Voltage Controlled Filter (MS-20 style)"
- note added: "Volume"
- note added: "Wet/Dry control"
- moved on the sheet: C101, C102, C103, C107, D101, D102, Q101, Q102, R101, R102, R103, R104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

Commit message: 4 layer layout
Parts:
- added C127: 22u, Capacitor_SMD:C_0805_2012Metric, symbol Device:C
- added TP107: GG, TestPoint:TestPoint_THTPad_D2.0mm_Drill1.0mm_VAL, symbol Connector:TestPoint
- added TP109: +9, TestPoint:TestPoint_THTPad_D2.0mm_Drill1.0mm_VAL, symbol Connector:TestPoint
- added TP110: -9, TestPoint:TestPoint_THTPad_D2.0mm_Drill1.0mm_VAL, symbol Connector:TestPoint
- TP103: value HP -> CE
- TP104: value LP -> WET
Connections:
- net HP_OUT is gone; now on net ComEmmiter: TP103.1
- net LP_OUT is gone; now on net WET: TP104.1
- net +9V: now also C127.1, TP109.1
- net -9V: now also TP110.1
- net EnvNeg: now also U102.7; no longer U102.1
- net EnvPos: now also U101.14, U102.10 (+); no longer U101.7, U102.6 (-)
- net FullRect: now also U101.10 (+), U101.7; no longer U101.1, U101.12 (+)
- net GND: now also U101.5 (+), U102.12 (+), U102.5 (+), C127.2; no longer U101.10 (+), U102.3 (+), U103.9 (-)
- net GTR_GAIN: now also U103.7, TP107.1; no longer U102.8
- net at C117.2, D105.2 (A), D106.1 (K)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: now also U103.8; no longer U103.7
- net at C110.1, R124.2: now also U101.12 (+); no longer U101.5 (+)
- net at R108.1, R109.1: now also U101.13 (-); no longer U101.6 (-)
- net at D101.2 (A), D102.1 (K): now also U101.1; no longer U101.8
- net at Q103.1 (B): now also U102.8; no longer U102.7
- net at Q103.2 (E), R119.1: now also U102.9 (-); no longer U102.5 (+)
- net at R140.2, RV105.3: now also U102.1; no longer U102.14
- net at D105.1 (K), D106.2 (A), D109.1 (K)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: now also U103.9 (-); no longer U103.6 (-)
- net at C104.1, R106.2, R107.1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: now also U101.9 (-); no longer U101.13 (-)
- net at D103.2 (A): now also U101.8; no longer U101.14
- net at R101.2, R102.2, R103.1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: now also U101.6 (-); no longer U101.2 (-)
- net at R122.1, R123.1: now also U103.6 (-); no longer U102.9 (-)
- net at D101.1 (K), R104.2, R105.1: now also U101.2 (-); no longer U101.9 (-)
- net at R137.2, R138.1: now also U102.3 (+); no longer U102.12 (+)
- net at R139.2, R140.1: now also U102.2 (-); no longer U102.13 (-)
- net at C107.2, Q102.3 (C), R115.1: now also U102.13 (-); no longer U103.10 (+)
- net at C109.2, R121.1: now also U103.5 (+); no longer U102.10 (+)
- net at C107.1, R116.2: now also U102.14; no longer U103.8
- net at RV101.2: now also U103.10 (+); no longer U103.5 (+)
- net at R117.2, R118.1: now also U102.6 (-); no longer U102.2 (-)
Other:
- moved on the sheet: C109, C110, C111, C112, C113, C114, C115, C116, C117, C121, D105, D106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

Commit message: rev2 gerber
Parts:
- added TP111: LP1, TestPoint:TestPoint_THTPad_D2.0mm_Drill1.0mm_VAL, symbol Connector:TestPoint
- added TP112: LP2, TestPoint:TestPoint_THTPad_D2.0mm_Drill1.0mm_VAL, symbol Connector:TestPoint
- added TP113: FB, TestPoint:TestPoint_THTPad_D2.0mm_Drill1.0mm_VAL, symbol Connector:TestPoint
Connections:
- net LP1: now reaches C117.1, U103.3 (+), U104.12
- net LP1: now also TP111.1
- net Feedback: now reaches C117.2, D105.2 (A), D106.1 (K), D109.2 (A), D110.1 (K), R135.1, U103.8
- net Feedback: now also TP113.1
- net LP2: now reaches C116.1, U103.12 (+), U104.5
- net LP2: now also TP112.1
Other:
- moved on the sheet: TP103, TP104, TP105, TP106, TP107, TP108, TP109, TP110
