File: EnvFilterPedal.kicad_sch (KiCad schematic)
At the start: 111 parts, among them J1 ScopeGroundLoop, J2 IO, Q1 BC847, Q2 BC857, Q3 BC857, U1 TL074, U2 TL074, U3 TL074, U4 LM13700, U5 AZ34063U

Commit message: rev5 routed & drc passing
Parts:
- removed C17, C21, C24: 220u, Capacitor_THT:CP_Radial_D5.0mm_P2.00mm, symbol Device:C_Polarized_US
- removed C20: 470p, Capacitor_SMD:C_0805_2012Metric, symbol Device:C
- removed C22: 470u, Capacitor_THT:CP_Radial_D5.0mm_P2.00mm, symbol Device:C_Polarized_US
- removed C26: 10u, Capacitor_SMD:C_0805_2012Metric, symbol Device:C
- removed D7: PMEG3030, Diode_SMD:D_SOD-123, symbol Device:D_Schottky
- removed L2: 4u7, Inductor_SMD:L_Bourns_SRP3212, symbol Device:L
- removed R37: 0.24R, Resistor_SMD:R_0805_2012Metric, symbol Device:R_US
- removed R40: 51k, Resistor_SMD:R_0805_2012Metric, symbol Device:R_US
- removed R41: 8k2, Resistor_SMD:R_0805_2012Metric, symbol Device:R_US
- removed TP14: -9R, TestPoint:TestPoint_THTPad_D2.0mm_Drill1.0mm_VAL, symbol Connector:TestPoint
- removed U5: AZ34063U, Package_SO:SO-8_3.9x4.9mm_P1.27mm, symbol Regulator_Switching:AZ34063U
- added C122: 100p, Capacitor_SMD:C_0805_2012Metric, symbol Device:C
- added C123: 4u7, Capacitor_SMD:C_0805_2012Metric, symbol Device:C
- added C124: 2u2, Capacitor_SMD:C_0805_2012Metric, symbol Device:C
- added C125: 100u, Capacitor_THT:CP_Radial_D5.0mm_P2.00mm, symbol Device:C_Polarized_US
- added D1: SS1060FL, Diode_SMD:D_SOD-123F, symbol Device:D_Schottky
- added NT1: NetTie_2, NetTie:NetTie-2_SMD_Pad0.5mm, symbol Device:NetTie_2
- added R144: 300k, Resistor_SMD:R_0805_2012Metric, symbol Device:R_US
- added R145: 22k, Resistor_SMD:R_0805_2012Metric, symbol Device:R_US
- added R146: 47k, Resistor_SMD:R_0805_2012Metric, symbol Device:R_US
- added U1: LMR62014XMF, Package_TO_SOT_SMD:SOT-23-5, symbol Regulator_Switching:LMR62014XMF
- C103: renamed from C5; value 100n -> 1u
- J101: renamed from J1; footprint Connector_Pin:THT_GND_WIRE -> Connector:THT_GND_WIRE
- L1: value 68uH -> 10u; footprint Inductor_SMD:L_TDK_VLS6045EX_VLS6045AF -> Inductor_SMD:L_SigTransformer_SLPPI04_15
- R102: renamed from R10; value 47k -> 100k
- RV101: renamed from RV3; footprint Potentiometer_THT:Potentiometer_Alpha_RV16AF_42_Single_Long -> Potentiometer_THT:Potentiometer_Alpha_RV16AF_42_VeryLong
- RV102: renamed from RV2; footprint Potentiometer_THT:Potentiometer_Alpha_RV16AF_42_Single_Long -> Potentiometer_THT:Potentiometer_Alpha_RV16AF_42_VeryLong
- RV103: renamed from RV1; footprint Potentiometer_THT:Potentiometer_Alpha_RV16AF_42_Single_Long -> Potentiometer_THT:Potentiometer_Alpha_RV16AF_42_VeryLong
- RV104: renamed from RV4; footprint Potentiometer_THT:Potentiometer_Alpha_RV16AF_42_Single_Long -> Potentiometer_THT:Potentiometer_Alpha_RV16AF_42_VeryLong
- RV105: renamed from RV5; footprint Potentiometer_THT:Potentiometer_Alpha_RV16AF_42_Single_Long -> Potentiometer_THT:Potentiometer_Alpha_RV16AF_42_VeryLong
- renumbered C2 to C101, C1 to C102, C11 to C104, C3 to C106, C16 to C107, C4 to C108, C6 to C109, C13 to C110, C7 to C111, C8 to C112, C12 to C113, C9 to C114, C10 to C115, C15 to C116, C14 to C117, C18 to C118, C19 to C119, C23 to C120, C25 to C121, D1 to D101, D2 to D102, D3 to D103, D6 to D104, D8 to D108, D4 to D109, D5 to D110, J2 to J102, Q3 to Q101, Q2 to Q102, Q1 to Q103, R14 to R103, R1 to R104, R5 to R105, R8 to R106, R12 to R107, R21 to R108, R20 to R109, R30 to R110, R31 to R111, R32 to R112, R33 to R113, R34 to R114, R35 to R115, R36 to R116, R3 to R117, R7 to R118, R25 to R119, R11 to R120, R2 to R121, R6 to R122, R4 to R123, R16 to R124, R15 to R125, R17 to R126, R13 to R127, R18 to R128, R24 to R129, R27 to R130, R23 to R131, R28 to R132, R19 to R133, R29 to R134, R22 to R135, R26 to R136, R43 to R137, R44 to R138, R42 to R139, R45 to R140, R38 to R141, R39 to R142, R46 to R143, R47 to R154, TP2 to TP101, TP4 to TP102, TP8 to TP103, TP9 to TP104, TP10 to TP105, TP11 to TP106, TP6 to TP107, TP5 to TP108, TP12 to TP109, TP13 to TP110, TP1 to TP111, TP3 to TP112, TP7 to TP113, U1 to U101, U2 to U102, U3 to U103, U4 to U104
Connections:
- net +9V: now also C122.2, C123.1, D1.1 (K), R144.2; no longer J102.5 (Pin_5)
- net -9V: now also J101.1, J102.4 (Pin_4), C123.2, C124.2, C125.2, R145.1, U1.2 (GND)
- net GND: now also C125.1, NT1.1; no longer J101.1, J102.4 (Pin_4), L1.2
- net GTR_GAIN: now also U102.1; no longer U103.7
- net at R140.2, RV105.3: now also U103.7; no longer U102.1
- net at R122.1, R123.1: now also U102.2 (-); no longer U103.6 (-)
- net at C109.2, R121.1: now also U102.3 (+); no longer U103.5 (+)
- net at R139.2, R140.1: now also U103.6 (-); no longer U102.2 (-)
- net at R137.2, R138.1: now also U103.5 (+); no longer U102.3 (+)
- net SWE renamed VCC
- net VCC: now also J102.5 (Pin_5), C124.1, NT1.2, R146.1, U1.5 (VIN)
- new net: D1.2 (A), L1.2, U1.1 (SW)
- new net: C122.1, R144.1, R145.2, U1.3 (FB)
- new net: R146.2, U1.4 (EN)
Other:
- note added: "Boost Converter"
- note removed: "Inverting SMPS"
- moved on the sheet: C121, D108, D109, D110, J102, R154, U102A, U103B
